File: Self Balancing robot/Self Balancing robot.kicad_sch (KiCad schematic)
At the start: 12 parts, among them J1 TB002-500-02BE, J2 691137710003, J3 691137710003, J4 691137710003, J5 TB002-500-03BE, J6 SSK01-MPH-254-A4, J7 SSK01-MPH-254-A4, U1 ESP32-DEVKIT-V1

Commit message: Initialize repo
Parts:
- removed BT1: Battery_Cell, symbol Device:Battery_Cell
- removed J2, J3, J4: 691137710003, 691137710003:691137710003, symbol 3 terminal block:691137710003
- removed J6: SSK01-MPH-254-A4, 4 pin male header:SAMESKY_SSK01-MPH-254-A4, symbol 4 pin male header:SSK01-MPH-254-A4
- removed MPU1: (no value), symbol MPU6050:MPU6050
- added J2, J3: (no value), Max7219:Max7219 Footprint, symbol Max7219 Sym:PPTC051LFBN-RC
- added J4: (no value), 5 pin male header:5 pin male header, symbol 5 pin male header:PPTC051LFBN-RC
- added J6: (no value), 5 V Buck Converter:5V buck converter, symbol 5V buck Converter:PPTC051LFBN-RC
- added J8: SSK01-MPH-254-A4, 4 pin male header:SAMESKY_SSK01-MPH-254-A4, symbol 4 pin male header:SSK01-MPH-254-A4
- added U2: GY-521, MPU 6050:MODULE_GY-521, symbol MPU 6050:GY-521
- U1: footprint ESP32 DevKitv1:MODULE_ESP32_DEVKIT_V1 -> ESP32_DEVKIT_V1_Files:MODULE_ESP32_DEVKIT_V1
Connections:
- net +5V: now also U1.30 (VIN), J2.1 (VIN), J6.1 (OUT+), U2.VCC
- net +7.5V: now also J6.4 (IN+)
- net GND: now also J1.2, J5.1, J2.2 (GND), J6.2 (OUT-), J6.3 (IN-), U2.GND
- net at A2.3 (1B): now also J8.1
- net at A2.4 (1A): now also J8.3
- net at A2.5 (2A): now also J8.2
- net at A2.6 (2B): now also J8.4
- net at U1.14 (D22): now also U2.SCL
- net at U1.11 (D21): now also U2.SDA
- net at U1.15 (D23): now also J2.3 (DIN)
- net at U1.8 (D5): now also J2.4 (CS)
- net at U1.9 (D18): now also J2.5 (CLK)
- new net: J3.1 (VIN), J4.1
- new net: J3.2 (GND), J4.2
- new net: J3.3 (DIN), J4.3
- new net: J3.4 (CS), J4.4
- new net: J3.5 (CLK), J4.5

Commit message: Updated PCB board
Parts:
- added C1, C2: C, Capacitor_THT:CP_Radial_D10.0mm_P5.00mm, symbol Device:C
Connections:
- net +7.5V: now also C1.1, C2.1
- net GND: now also C1.2, C2.2

Commit message: In progress commit (Will fix on laptop)
Parts:
- added U?: (no value), 5A Fuse:5A Fuse, symbol 5A Fuse:5A Fuse
Connections:
- net +7.5V: now also U?.2 (Output); no longer J5.3
- new net: J5.3, U?.1 (Input)
Changed lines of the file:
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@@
 	(wire
 		(pts
-			(xy 63.5 31.75) (xy 71.12 31.75)
+			(xy 39.37 41.91) (xy 39.37 40.64)
 		)
 		(stroke
@@
 	(wire
 		(pts
-			(xy 59.69 34.29) (xy 63.5 34.29)
-		)
-		(stroke
-			(width 0)
-			(type default)
-		)
-	)
-	(wire
-		(pts
 			(xy 27.94 161.29) (xy 113.03 161.29)
 		)
@@
 	(wire
 		(pts
-			(xy 69.85 41.91) (xy 69.85 40.64)
-		)
-		(stroke
-			(width 0)
-			(type default)
-		)
-	)
-	(wire
-		(pts
 			(xy 223.52 80.01) (xy 223.52 60.96)
 		)
@@
 	(wire
 		(pts
+			(xy 46.99 35.56) (xy 46.99 38.1)
+		)
+		(stroke
+			(width 0)
+			(type default)
+		)
+	)
+	(wire
+		(pts
 			(xy 158.75 93.98) (xy 158.75 95.25)
 		)
@@
 	(wire
 		(pts
+			(xy 39.37 41.91) (xy 69.85 41.91)
+		)
+		(stroke
+			(width 0)
+			(type default)
+		)
+	)
+	(wire
+		(pts
 			(xy 152.4 55.88) (xy 152.4 62.23)
 		)
@@
 	(wire
 		(pts
-			(xy 63.5 34.29) (xy 63.5 31.75)
+			(xy 71.12 31.75) (xy 71.12 38.1)
 		)
 		(stroke
@@
 	(wire
 		(pts
-			(xy 69.85 40.64) (xy 66.04 40.64)
-		)
-		(stroke
-			(width 0)
-			(type default)
-		)
-	)
-	(wire
-		(pts
 			(xy 30.48 93.98) (xy 24.13 93.98)
 		)
@@
 	(wire
 		(pts
+			(xy 46.99 38.1) (xy 48.26 38.1)
+		)
+		(stroke
+			(width 0)
+			(type default)
+		)
+	)
+	(wire
+		(pts
 			(xy 40.64 111.76) (xy 40.64 115.57)
 		)
@@
 		(pts
 			(xy 152.4 62.23) (xy 123.19 62.23)
+		)
+		(stroke
+			(width 0)
+			(type default)
+		)
+	)
+	(wire
+		(pts
+			(xy 71.12 38.1) (xy 67.31 38.1)
 		)
 		(stroke
@@
 	(symbol
 		(lib_id "power:+7.5V")
-		(at 59.69 34.29 0)
+		(at 46.99 35.56 0)
 		(unit 1)
 		(body_style 1)
@@
 		(fields_autoplaced yes)
 		(property "Reference" "#PWR01"
-			(at 59.69 38.1 0)
+			(at 46.99 39.37 0)
 			(hide yes)
 			(show_name no)
@@
 		)
 		(property "Value" "+7.5V"
-			(at 59.69 29.21 0)
+			(at 46.99 30.48 0)
 			(show_name no)
 			(do_not_autoplace no)
@@
 		)
 		(property "Footprint" ""
-			(at 59.69 34.29 0)
+			(at 46.99 35.56 0)
 			(hide yes)
 			(show_name no)
@@
 		)
 		(property "Datasheet" ""
-			(at 59.69 34.29 0)
+			(at 46.99 35.56 0)
 			(hide yes)
 			(show_name no)
@@
 		)
 		(property "Description" "Power symbol creates a global label with name \"+7.5V\""
-			(at 59.69 34.29 0)
+			(at 46.99 35.56 0)
 			(hide yes)
 			(show_name no)
@@
 	)
 	(symbol
+		(lib_id "5A Fuse:5A Fuse")
+		(at 62.23 41.91 180)
+		(unit 1)
+		(body_style 1)
+		(exclude_from_sim no)
+		(in_bom yes)
+		(on_board yes)
+		(in_pos_files yes)
+		(dnp no)
+		(fields_autoplaced yes)
+		(property "Reference" "U?"
+			(at 57.785 34.29 0)
+			(show_name no)
+			(do_not_autoplace no)
+			(effects
+				(font
+					(size 1.27 1.27)
+				)
+			)
+		)
+		(property "Value" ""
+			(at 62.23 41.91 0)
+			(show_name no)
+			(do_not_autoplace no)
+			(effects
+				(font
+					(size 1.27 1.27)
+				)
+			)
+		)
+		(property "Footprint" "5A Fuse:5A Fuse"
+			(at 62.23 41.91 0)
+			(hide yes)
+			(show_name no)
+			(do_not_autoplace no)
+			(effects
+				(font
+					(size 1.27 1.27)
+				)
+			)
+		)
+		(property "Datasheet" ""
+			(at 62.23 41.91 0)
+			(hide yes)
+			(show_name no)
+			(do_not_autoplace no)
+			(effects
+				(font
+					(size 1.27 1.27)
+				)
+			)
+		)
+		(property "Description" ""
+			(at 62.23 41.91 0)
+			(hide yes)
+			(show_name no)
+			(do_not_autoplace no)
+			(effects
+				(font
+					(size 1.27 1.27)
+				)
+			)
+		)
+		(pin "2"
+		)
+		(pin "1"
+		)
+		(instances
+			(project "Self Balancing robot"
+				(path "/065b4eff-ee6e-40f5-afb6-a69d6586b899"
+					(reference "U?")
+					(unit 1)
+				)
+			)
+		)
+	)
+	(symbol
 		(lib_id "power:GND")
 		(at 64.77 44.45 0)
@@
 	(symbol
 		(lib_id "power:+7.5V")
-		(at 66.04 40.64 0)
+		(at 39.37 40.64 0)
 		(unit 1)
 		(body_style 1)
@@
 		(fields_autoplaced yes)
 		(property "Reference" "#PWR02"
-			(at 66.04 44.45 0)
+			(at 39.37 44.45 0)
 			(hide yes)
 			(show_name no)
@@
 		)
 		(property "Value" "+7.5V"
-			(at 66.04 35.56 0)
+			(at 39.37 35.56 0)
 			(show_name no)
 			(do_not_autoplace no)
@@
 		)
 		(property "Footprint" ""
-			(at 66.04 40.64 0)
+			(at 39.37 40.64 0)
 			(hide yes)
 			(show_name no)
@@
 		)
 		(property "Datasheet" ""
-			(at 66.04 40.64 0)
+			(at 39.37 40.64 0)
 			(hide yes)
 			(show_name no)
@@
 		)
 		(property "Description" "Power symbol creates a global label with name \"+7.5V\""
-			(at 66.04 40.64 0)
-			(hide yes)
-			(show_name no)
+			(at 39.37 40.64 0)
+			(hide yes)
+			(show_name no)

Commit message: Final Commit. PCB Finished!
Parts:
- added R1: R, Resistor_THT:R_Axial_DIN0207_L6.3mm_D2.5mm_P15.24mm_Horizontal, symbol Device:R
- gave numbers to parts that had none: 1
Connections:
- net +7.5V: now also R1.1; no longer J1.1
- net GND: no longer J5.1
- new net: J1.1, R1.2
Other:
- moved on the sheet: U3
Changed lines of the file:
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@@
+	(wire
+		(pts
+			(xy 39.37 41.91) (xy 48.26 41.91)
+		)
+		(stroke
+			(width 0)
+			(type default)
+		)
+	)
 	(wire
 		(pts
@@
 	(wire
 		(pts
-			(xy 46.99 35.56) (xy 46.99 38.1)
+			(xy 31.75 29.21) (xy 31.75 31.75)
 		)
 		(stroke
@@
 	(wire
 		(pts
-			(xy 39.37 41.91) (xy 69.85 41.91)
-		)
-		(stroke
-			(width 0)
-			(type default)
-		)
-	)
-	(wire
-		(pts
 			(xy 152.4 55.88) (xy 152.4 62.23)
 		)
@@
 	(wire
 		(pts
-			(xy 49.53 25.4) (xy 71.12 25.4)
-		)
-		(stroke
-			(width 0)
-			(type default)
-		)
-	)
-	(wire
-		(pts
 			(xy 76.2 58.42) (xy 76.2 133.35)
 		)
@@
 	(wire
 		(pts
-			(xy 71.12 31.75) (xy 71.12 38.1)
-		)
-		(stroke
-			(width 0)
-			(type default)
-		)
-	)
-	(wire
-		(pts
 			(xy 139.7 76.2) (xy 139.7 77.47)
 		)
@@
 	(wire
 		(pts
+			(xy 55.88 41.91) (xy 69.85 41.91)
+		)
+		(stroke
+			(width 0)
+			(type default)
+		)
+	)
+	(wire
+		(pts
 			(xy 20.32 168.91) (xy 124.46 168.91)
 		)
@@
 	(wire
 		(pts
-			(xy 46.99 38.1) (xy 48.26 38.1)
+			(xy 31.75 31.75) (xy 35.56 31.75)
 		)
 		(stroke
@@
 	(wire
 		(pts
-			(xy 71.12 38.1) (xy 67.31 38.1)
+			(xy 54.61 31.75) (xy 71.12 31.75)
 		)
 		(stroke
@@
 		(pts
 			(xy 139.7 114.3) (xy 139.7 118.11)
-		)
-		(stroke
-			(width 0)
-			(type default)
-		)
-	)
-	(wire
-		(pts
-			(xy 71.12 25.4) (xy 71.12 26.67)
 		)
 		(stroke
@@
 	(symbol
 		(lib_id "power:+7.5V")
-		(at 46.99 35.56 0)
+		(at 31.75 29.21 0)
 		(unit 1)
 		(body_style 1)
@@
 		(fields_autoplaced yes)
 		(property "Reference" "#PWR01"
-			(at 46.99 39.37 0)
+			(at 31.75 33.02 0)
 			(hide yes)
 			(show_name no)
@@
 		)
 		(property "Value" "+7.5V"
-			(at 46.99 30.48 0)
+			(at 31.75 24.13 0)
 			(show_name no)
 			(do_not_autoplace no)
@@
 		)
 		(property "Footprint" ""
-			(at 46.99 35.56 0)
+			(at 31.75 29.21 0)
 			(hide yes)
 			(show_name no)
@@
 		)
 		(property "Datasheet" ""
-			(at 46.99 35.56 0)
+			(at 31.75 29.21 0)
 			(hide yes)
 			(show_name no)
@@
 		)
 		(property "Description" "Power symbol creates a global label with name \"+7.5V\""
-			(at 46.99 35.56 0)
+			(at 31.75 29.21 0)
 			(hide yes)
 			(show_name no)
@@
 	(symbol
 		(lib_id "5A Fuse:5A Fuse")
-		(at 62.23 41.91 180)
+		(at 49.53 35.56 180)
 		(unit 1)
 		(body_style 1)
@@
 		(dnp no)
 		(fields_autoplaced yes)
-		(property "Reference" "U?"
-			(at 57.785 34.29 0)
+		(property "Reference" "U3"
+			(at 45.085 27.94 0)
 			(show_name no)
 			(do_not_autoplace no)
@@
 		)
 		(property "Value" ""
-			(at 62.23 41.91 0)
+			(at 49.53 35.56 0)
 			(show_name no)
 			(do_not_autoplace no)
@@
 		)
 		(property "Footprint" "5A Fuse:5A Fuse"
-			(at 62.23 41.91 0)
+			(at 49.53 35.56 0)
 			(hide yes)
 			(show_name no)
@@
 		)
 		(property "Datasheet" ""
-			(at 62.23 41.91 0)
+			(at 49.53 35.56 0)
 			(hide yes)
 			(show_name no)
@@
 		)
 		(property "Description" ""
-			(at 62.23 41.91 0)
+			(at 49.53 35.56 0)
 			(hide yes)
 			(show_name no)
@@
 			(project "Self Balancing robot"
 				(path "/065b4eff-ee6e-40f5-afb6-a69d6586b899"
-					(reference "U?")
+					(reference "U3")
 					(unit 1)
 				)
@@
 	)
 	(symbol
-		(lib_id "power:GND")
-		(at 49.53 25.4 0)
+		(lib_id "Device:R")
+		(at 52.07 41.91 90)
 		(unit 1)
 		(body_style 1)
@@
 		(dnp no)
 		(fields_autoplaced yes)
-		(property "Reference" "#PWR014"
-			(at 49.53 31.75 0)
-			(hide yes)
-			(show_name no)
-			(do_not_autoplace no)
-			(effects
-				(font
-					(size 1.27 1.27)
-				)
-			)
-		)
-		(property "Value" "GND"
-			(at 49.53 30.48 0)
-			(show_name no)
-			(do_not_autoplace no)
-			(effects
-				(font
-					(size 1.27 1.27)
-				)
-			)
-		)
-		(property "Footprint" ""
-			(at 49.53 25.4 0)
+		(property "Reference" "R1"
+			(at 52.07 35.56 90)
+			(show_name no)
+			(do_not_autoplace no)
+			(effects
+				(font
+					(size 1.27 1.27)
+				)
+			)
+		)
+		(property "Value" "R"
+			(at 52.07 38.1 90)
+			(show_name no)
+			(do_not_autoplace no)
+			(effects
+				(font
+					(size 1.27 1.27)
+				)
+			)
+		)
+		(property "Footprint" "Resistor_THT:R_Axial_DIN0207_L6.3mm_D2.5mm_P15.24mm_Horizontal"
+			(at 52.07 43.688 90)
 			(hide yes)
 			(show_name no)
@@
 		)
 		(property "Datasheet" ""
-			(at 49.53 25.4 0)
-			(hide yes)
-			(show_name no)
-			(do_not_autoplace no)
-			(effects
-				(font
-					(size 1.27 1.27)
-				)
-			)
-		)
-		(property "Description" "Power symbol creates a global label with name \"GND\" , ground"
-			(at 49.53 25.4 0)
+			(at 52.07 41.91 0)
+			(hide yes)
+			(show_name no)
+			(do_not_autoplace no)
+			(effects
+				(font
+					(size 1.27 1.27)
+				)
+			)
+		)
+		(property "Description" "Resistor"
+			(at 52.07 41.91 0)
 			(hide yes)
 			(show_name no)
@@
 		)
 		(pin "1"
+		)
+		(pin "2"
 		)
 		(instances
 			(project "Self Balancing robot"
 				(path "/065b4eff-ee6e-40f5-afb6-a69d6586b899"
-					(reference "#PWR014")
+					(reference "R1")
 					(unit 1)
 				)
