File: Self Balancing robot/Self Balancing robot.kicad_pcb (KiCad board)
At the start: 2 copper layers, 4 parts, among them J1 TB002-500-02BE, J5 TB002-500-03BE, J6 SSK01-MPH-254-A4, U1 ESP32-DEVKIT-V1

Commit message: Initialize repo
Parts:
- added A1: Pololu_Breakout_A4988, Module:Pololu_Breakout-16_15.2x20.3mm, F.Cu at (111.6, 39.5)
- added A2: Pololu_Breakout_A4988, Module:Pololu_Breakout-16_15.2x20.3mm, F.Cu at (128.3, 39.5)
- added J2: ~, Max7219:Max7219 Footprint, F.Cu at (4.06, 16.9)
- added J3: ~, Max7219:Max7219 Footprint, F.Cu at (4.06, 22.0)
- added J4: ~, 5 pin male header:5 pin male header, F.Cu at (4.06, 27.2)
- added J7: SSK01-MPH-254-A4, 4 pin male header:SAMESKY_SSK01-MPH-254-A4, F.Cu at (132.9, 61.4)
- added J8: SSK01-MPH-254-A4, 4 pin male header:SAMESKY_SSK01-MPH-254-A4, F.Cu at (132.9, 65.4)
- added U2: GY-521, MPU 6050:MODULE_GY-521, F.Cu at (118.1, 70.3)
- J6: value SSK01-MPH-254-A4 -> ~; footprint 4 pin male header:SAMESKY_SSK01-MPH-254-A4 -> 5 pin male header:5 pin male header
- U1: footprint ESP32 DevKitv1:MODULE_ESP32_DEVKIT_V1 -> ESP32_DEVKIT_V1_Files:MODULE_ESP32_DEVKIT_V1
- moved J6 57.2 mm to (39.5, 107.6)
Connections:
- J1 pad 2: unconnected-(J1-Pad2) -> GND
- J5 pad 1: unconnected-(J5-Pad1) -> GND
- J6 pad 1: unconnected-(J6-Pad1) -> +5V
- J6 pad 2: unconnected-(J6-Pad2) -> GND
- J6 pad 3: unconnected-(J6-Pad3) -> GND
- J6 pad 4: unconnected-(J6-Pad4) -> +7.5V
- U1 pad 11: unconnected-(U1-D21-Pad11) -> Net-(U1-D21)
- U1 pad 14: unconnected-(U1-D22-Pad14) -> Net-(U1-D22)
- U1 pad 15: unconnected-(U1-D23-Pad15) -> Net-(J2-3)
- U1 pad 23: unconnected-(U1-D25-Pad23) -> Net-(A2-DIR)
- U1 pad 24: unconnected-(U1-D26-Pad24) -> Net-(A2-STEP)
- U1 pad 30: unconnected-(U1-VIN-Pad30) -> +5V
- U1 pad 6: unconnected-(U1-RX2-Pad6) -> Net-(A1-DIR)
- U1 pad 7: unconnected-(U1-TX2-Pad7) -> Net-(A1-STEP)
- U1 pad 8: unconnected-(U1-D5-Pad8) -> Net-(J2-1)
- U1 pad 9: unconnected-(U1-D18-Pad9) -> Net-(J2-4)

Commit message: Updated PCB board
Parts:
- added C1: C, Capacitor_THT:CP_Radial_D10.0mm_P5.00mm, F.Cu at (106.8, 117.0)
- added C2: C, Capacitor_THT:CP_Radial_D10.0mm_P5.00mm, F.Cu at (149.5, 116.3)
- A1, A2, J7, J8, U1: moved to B.Cu
- J6: footprint 5 pin male header:5 pin male header -> 5 V Buck Converter:5V buck converter
- moved J2 213.1 mm to (162.0, 160.0)
- moved J4 157.7 mm to (89.0, 160.0)
- moved J3 155.7 mm to (89.0, 152.5)
- moved J5 138.1 mm to (167.5, 154.0), turned to 90 degrees
- moved J1 110.5 mm to (167.3, 136.5), turned to 90 degrees
- moved A2 80.6 mm to (172.3, 107.1), turned to 180 degrees
- moved A1 68.4 mm to (100.8, 107.1), turned to 180 degrees
- moved U2 67.7 mm to (130.1, 136.9)
- moved J7 66.9 mm to (94.2, 116.0), turned to -90 degrees
- moved J8 60.5 mm to (166.5, 115.7), turned to -90 degrees
- moved J6 56.6 mm to (85.5, 140.6)
- moved U1 32.7 mm to (130.5, 135.0)
Routing:
- net GND: track 0.00 -> 303.8 mm
- net +7.5V: track 0.00 -> 193.2 mm
- net +5V: track 0.00 -> 184.1 mm
- net Net-(J2-DIN): track 0.00 -> 75.6 mm
- net Net-(A1-DIR): track 0.00 -> 71.2 mm
- net Net-(J2-CLK): track 0.00 -> 69.8 mm
- net Net-(J2-CS): track 0.00 -> 64.0 mm
- net Net-(A1-STEP): track 0.00 -> 45.4 mm
- net Net-(A2-STEP): track 0.00 -> 42.2 mm
- net Net-(A2-DIR): track 0.00 -> 39.3 mm
- net Net-(U1-D22): track 0.00 -> 18.1 mm
- net Net-(U1-D21): track 0.00 -> 13.0 mm
- net Net-(A1-2A): track 0.00 -> 7.70 mm
- net Net-(A1-1A): track 0.00 -> 7.70 mm
- net Net-(A2-2A): track 0.00 -> 7.00 mm
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Other:
- board outline added: 90 x 60 mm
- board text added: "+"

Commit message: Updates
Parts:
- moved J6 4.51 mm to (84.0, 136.4)
Routing:
- net +7.5V: track 193.2 -> 164.5 mm
- net +5V: track 184.1 -> 180.4 mm
- net GND: track 303.8 -> 301.6 mm
Other:
- board text removed: "+"

Commit message: In progress commit (Will fix on laptop)
Parts:
- added U3: ~, 5A Fuse:5A Fuse, F.Cu at (170.2, 118.4)
- A1, A2: moved to F.Cu
- moved J7 15.6 mm to (109.3, 112.2)
- moved U2 14.8 mm to (144.3, 132.9)
- moved J3 14.8 mm to (103.2, 148.5)
- moved J4 14.8 mm to (103.2, 156.0)
- moved J6 14.8 mm to (98.2, 132.3)
- moved C1 14.8 mm to (121.0, 113.0)
- moved C2 14.8 mm to (163.7, 112.2)
- moved J8 14.8 mm to (180.7, 111.7)
- moved J1 14.8 mm to (181.5, 132.5)
- moved J2 14.8 mm to (176.2, 156.0)
- moved J5 14.8 mm to (181.7, 150.0)
- moved U1 14.8 mm to (144.7, 131.0)
- moved A1 5.17 mm to (102.2, 102.1), turned to 0 degrees
- moved A2 4.76 mm to (174.4, 102.8), turned to 0 degrees
Connections:
- J5 pad 3: +7.5V -> Net-(U3-Input)
Routing:
- net Net-(U3-Input): track 0.00 -> 18.4 mm
- net Net-(A2-DIR): track 39.3 -> 53.6 mm
- net Net-(A2-STEP): track 42.2 -> 55.4 mm
- net Net-(A1-STEP): track 45.4 -> 34.2 mm
- net +5V: track 180.4 -> 170.3 mm
- net GND: track 301.6 -> 309.3 mm
- net Net-(A2-2A): track 7.00 -> 0.00 mm
- net Net-(A2-1A): track 6.78 -> 0.00 mm
- net Net-(A2-2B): track 5.95 -> 0.00 mm
- net Net-(A2-1B): track 5.95 -> 0.00 mm
- net Net-(A1-2A): track 7.70 -> 13.3 mm
- net Net-(A2-~{RESET}): track 2.54 -> 0.00 mm
- net Net-(A1-~{RESET}): track 2.54 -> 0.00 mm
- net Net-(A1-1A): track 7.70 -> 8.71 mm
- net Net-(A1-2B): track 6.65 -> 7.66 mm
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Other:
- outline, holes or cut-outs redrawn

Commit message: Final Commit. PCB Finished!
Parts:
- moved A2 0.71 mm to (174.9, 102.4)
Routing:
- net +5V: track 170.3 -> 152.8 mm
- net GND: track 309.3 -> 321.7 mm
- net Net-(A2-1A): track 0.00 -> 7.03 mm
- net Net-(A2-2A): track 0.00 -> 6.66 mm
- net Net-(A2-1B): track 0.00 -> 5.97 mm
- net Net-(A2-2B): track 0.00 -> 5.97 mm
- net Net-(A2-~{RESET}): track 0.00 -> 2.54 mm
- net Net-(A2-DIR): track 53.6 -> 54.5 mm

Commit message: Updated PCB with resistor
Parts:
- added R1: R, Resistor_THT:R_Axial_DIN0207_L6.3mm_D2.5mm_P15.24mm_Horizontal, F.Cu at (104.6, 141.0)
- MPU 6050: renamed from U2; value GY-521 -> MPU6050
- moved Max7219 11.8 mm to (115.0, 156.0)
- moved Max7219 11.2 mm to (165.0, 156.0)
- moved J3 6.85 mm to (110.0, 148.3)
- moved Fuse 1.98 mm to (170.2, 120.3)
- renumbered A2 to A4988, A1 to A4988, U1 to ESP, U3 to Fuse, J2 to Max7219, J4 to Max7219, J5 to TBlock3, J1 to Tblock2
Connections:
- TBlock3 pad 1: GND -> unconnected-(J5-Pad1)
- Tblock2 pad 1: +7.5V -> Net-(J1-Pad1)
Routing:
- net Net-(J1-Pad1): track 0.00 -> 104.5 mm
- net +5V: track 152.8 -> 198.3 mm
- net Net-(A1-DIR): track 71.8 -> 40.2 mm
- net +7.5V: track 163.7 -> 195.3 mm
- net GND: track 321.7 -> 334.0 mm
- net Net-(J2-DIN): track 75.6 -> 64.4 mm
- net Net-(J2-CS): track 64.0 -> 52.8 mm
- net Net-(J2-CLK): track 69.8 -> 58.7 mm
- net Net-(J3-VIN): track 0.00 -> 9.77 mm
- net Net-(J3-GND): track 0.00 -> 9.77 mm
- net Net-(J3-DIN): track 0.00 -> 9.77 mm
- net Net-(J3-CS): track 0.00 -> 9.77 mm
- net Net-(J3-CLK): track 0.00 -> 9.77 mm
- net Net-(A1-~{RESET}): track 0.00 -> 2.54 mm
- net Net-(U3-Input): track 18.4 -> 20.3 mm
Other:
- outline, holes or cut-outs redrawn
- board text added: "Bat+"
- board text added: "Common"
- board text added: "LED+"
- board text added: "NC"
- board text added: "NO"
